File: Hardware/Mutteruhr V2.0 USB-B - H-Brigde L298 - USB UART LM2576-5/mutteruhr-Haus.brd (EAGLE design)
At the start: 46 parts, among them IC1 atmega168, IC2 LM2576-5, IC4 L298, IC5 MCP2200SOIC20, Q1 8MHz, Q2 12MHz

Commit message: Fehler an USB MCP2200 VDD gefixt. Verbindung Pin 1 - 17 getrennt
Connections:
- net N$24: no longer IC5.17
Routing:
- net N$24: track 55.4 -> 53.4 mm
Changed lines of the file:
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@@
 <?xml version="1.0" encoding="utf-8"?>
 <!DOCTYPE eagle SYSTEM "eagle.dtd">
-<eagle version="7.7.0">
+<eagle version="7.6.0">
 <drawing>
 <settings>
@@
 </signal>
 <signal name="N$24">
-<contactref element="IC5" pad="17"/>
-<wire x1="66.2775" y1="63.5" x2="68.2625" y2="63.5" width="0.6096" layer="16"/>
 <contactref element="C5" pad="1"/>
 <wire x1="51.1175" y1="59.69" x2="50.4825" y2="60.325" width="0.4064" layer="16"/>
