File: Hardware/Mutteruhr V2.0 USB-B - H-Brigde L298 - USB UART LM2576-5/mutteruhr-Haus.sch (EAGLE design)
At the start: 42 parts, among them IC1 atmega168, IC2 LM2576-5, IC4 L298, IC5 MCP2200SOIC20, Q1 8MHz, Q2 12MHz, X1 MKDSN1,5/2-5,08, X3 MKDSN1,5/2-5,08, X4 MKDSN1,5/4-5,08

Commit message: Fehler an USB MCP2200 VDD gefixt. Verbindung Pin 1 - 17 getrennt
Connections:
- net N$24: no longer IC5.VUSB
Changed lines of the file:
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@@
 <?xml version="1.0" encoding="utf-8"?>
 <!DOCTYPE eagle SYSTEM "eagle.dtd">
-<eagle version="7.7.0">
+<eagle version="7.6.0">
 <drawing>
 <settings>
@@
 <net name="N$24" class="0">
 <segment>
-<pinref part="IC5" gate="G$1" pin="VUSB"/>
-<wire x1="203.2" y1="96.52" x2="223.52" y2="96.52" width="0.1524" layer="91"/>
-<wire x1="223.52" y1="96.52" x2="223.52" y2="91.44" width="0.1524" layer="91"/>
 <wire x1="223.52" y1="91.44" x2="223.52" y2="88.9" width="0.1524" layer="91"/>
 <wire x1="223.52" y1="88.9" x2="236.22" y2="88.9" width="0.1524" layer="91"/>
@@
 <pinref part="IC5" gate="G$1" pin="VDD"/>
 <wire x1="203.2" y1="91.44" x2="223.52" y2="91.44" width="0.1524" layer="91"/>
-<junction x="223.52" y="91.44"/>
 <pinref part="X5" gate="G$1" pin="VBUS"/>
 </segment>
