File: Hardware/Mutteruhr V2.1 External USB-B - H-Brigde L298 - USB UART LM2576-5/USB-Board.brd (EAGLE design)
At the start: 39.9 x 48.5 mm, 16 parts, among them IC5 MCP2200SOIC20, Q2 12MHz

Commit message: Fehler an USB MCP2200 VDD gefixt. Verbindung Pin 1 - 17 getrennt
Connections:
- net N$24: no longer IC5.17
Routing:
- net N$24: track 50.8 -> 48.8 mm
Changed lines of the file:
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@@
 <?xml version="1.0" encoding="utf-8"?>
 <!DOCTYPE eagle SYSTEM "eagle.dtd">
-<eagle version="7.7.0">
+<eagle version="7.6.0">
 <drawing>
 <settings>
@@
 <grid distance="0.0125" unitdist="inch" unit="inch" style="lines" multiple="1" display="no" altdistance="0.025" altunitdist="inch" altunit="inch"/>
 <layers>
-<layer number="1" name="Top" color="4" fill="1" visible="no" active="yes"/>
-<layer number="16" name="Bottom" color="1" fill="1" visible="no" active="yes"/>
-<layer number="17" name="Pads" color="2" fill="1" visible="no" active="yes"/>
-<layer number="18" name="Vias" color="2" fill="1" visible="no" active="yes"/>
-<layer number="19" name="Unrouted" color="6" fill="1" visible="no" active="yes"/>
+<layer number="1" name="Top" color="4" fill="1" visible="yes" active="yes"/>
+<layer number="16" name="Bottom" color="1" fill="1" visible="yes" active="yes"/>
+<layer number="17" name="Pads" color="2" fill="1" visible="yes" active="yes"/>
+<layer number="18" name="Vias" color="2" fill="1" visible="yes" active="yes"/>
+<layer number="19" name="Unrouted" color="6" fill="1" visible="yes" active="yes"/>
 <layer number="20" name="Dimension" color="15" fill="1" visible="no" active="yes"/>
 <layer number="21" name="tPlace" color="7" fill="1" visible="yes" active="yes"/>
@@
 </signal>
 <signal name="N$24">
-<contactref element="IC5" pad="17"/>
 <contactref element="C5" pad="1"/>
 <contactref element="IC5" pad="1"/>
 <contactref element="X5" pad="VBUS"/>
-<wire x1="20.955" y1="60.245" x2="20.955" y2="62.23" width="0.6096" layer="16"/>
 <wire x1="20.955" y1="62.23" x2="19.6288" y2="62.23" width="0.6096" layer="16"/>
 <wire x1="19.6288" y1="62.23" x2="17.8" y2="64.0588" width="0.6096" layer="16"/>
