File: Hardware/Mutteruhr V2.1 External USB-B - H-Brigde L298 - USB UART LM2576-5/USB-Board.sch (EAGLE design)
At the start: 12 parts, among them IC5 MCP2200SOIC20, Q2 12MHz

Commit message: Fehler an USB MCP2200 VDD gefixt. Verbindung Pin 1 - 17 getrennt
Connections:
- net N$24: no longer IC5.VUSB
Changed lines of the file:
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@@
 <?xml version="1.0" encoding="utf-8"?>
 <!DOCTYPE eagle SYSTEM "eagle.dtd">
-<eagle version="7.7.0">
+<eagle version="7.6.0">
 <drawing>
 <settings>
@@
 <net name="N$24" class="0">
 <segment>
-<pinref part="IC5" gate="G$1" pin="VUSB"/>
-<wire x1="76.2" y1="53.34" x2="96.52" y2="53.34" width="0.1524" layer="91"/>
-<wire x1="96.52" y1="53.34" x2="96.52" y2="48.26" width="0.1524" layer="91"/>
 <wire x1="96.52" y1="48.26" x2="96.52" y2="45.72" width="0.1524" layer="91"/>
 <wire x1="96.52" y1="45.72" x2="109.22" y2="45.72" width="0.1524" layer="91"/>
@@
 <pinref part="IC5" gate="G$1" pin="VDD"/>
 <wire x1="76.2" y1="48.26" x2="96.52" y2="48.26" width="0.1524" layer="91"/>
-<junction x="96.52" y="48.26"/>
 <pinref part="X5" gate="G$1" pin="VBUS"/>
 </segment>
